Commit message: change robot design, complete ball chasing packing, redo robot design

File: Project2/my_robot/urdf/my_robot.xacro (robot description, xacro)
@@ -10,8 +10,8 @@
   </joint>
   <link name='chassis'>
-    <pose>0 0 0.1 0 0 0</pose>
+    <pose>0 0 0.2 0 0 0</pose>
     <inertial>
       <mass value="15.0"/>
-      <origin xyz="0.0 0 0" rpy=" 0 0 0"/>
+      <origin xyz="0 0 0" rpy=" 0 0 0"/>
       <inertia
           ixx="0.1" ixy="0" ixz="0"
@@ -23,5 +23,5 @@
       <origin xyz="0 0 0" rpy=" 0 0 0"/>
       <geometry>
-        <box size=".4 .2 .1"/>
+        <cylinder radius="0.15" length="0.3"/>
       </geometry>
     </collision>
@@ -29,15 +29,15 @@
       <origin xyz="0 0 0" rpy=" 0 0 0"/>
       <geometry>
-        <box size=".4 .2 .1"/>
+        <cylinder radius="0.15" length="0.3"/>
       </geometry>
     </visual>
     <collision name='back_caster_collision'>
-      <origin xyz="-0.15 0 -0.05" rpy=" 0 0 0"/>
+      <origin xyz="-0.1 0 -0.15" rpy=" 0 0 0"/>
       <geometry>
-        <sphere radius="0.0499"/>
+        <sphere radius="0.05"/>
       </geometry>
     </collision>
     <visual name='back_caster_visual'>
-      <origin xyz="-0.15 0 -0.05" rpy=" 0 0 0"/>
+      <origin xyz="-0.1 0 -0.15" rpy=" 0 0 0"/>
       <geometry>
         <sphere radius="0.05"/>
@@ -45,11 +45,11 @@
     </visual>
     <collision name='front_caster_collision'>
-      <origin xyz="0.15 0 -0.05" rpy=" 0 0 0"/>
+      <origin xyz="0.1 0 -0.15" rpy=" 0 0 0"/>
       <geometry>
-        <sphere radius="0.0499"/>
+        <sphere radius="0.05"/>
       </geometry>
     </collision>
     <visual name='front_caster_visual'>
-      <origin xyz="0.15 0 -0.05" rpy=" 0 0 0"/>
+      <origin xyz="0.1 0 -0.15" rpy=" 0 0 0"/>
       <geometry>
         <sphere radius="0.05"/>
@@ -61,5 +61,5 @@
 			<origin xyz="0 0 0" rpy="0 1.57 1.57"/>
 			<geometry>
-				<cylinder radius="0.1" length="0.05"/>
+				<cylinder radius="0.15" length="0.05"/>
 			</geometry>
 		</collision>
@@ -76,5 +76,5 @@
 				<origin xyz="0 0 0" rpy="0 1.57 1.57"/>
 			<geometry>
-				<cylinder radius="0.1" length="0.05"/>
+				<cylinder radius="0.15" length="0.05"/>
 			</geometry>
 		</visual>
@@ -84,5 +84,5 @@
 			<origin xyz="0 0 0" rpy="0 1.57 1.57"/>
 			<geometry>
-				<cylinder radius="0.1" length="0.05"/>
+				<cylinder radius="0.15" length="0.05"/>
 			</geometry>
 		</collision>
@@ -99,10 +99,10 @@
 				<origin xyz="0 0 0" rpy="0 1.57 1.57"/>
 			<geometry>
-				<cylinder radius="0.1" length="0.05"/>
+				<cylinder radius="0.15" length="0.05"/>
 			</geometry>
 		</visual>
 	</link>
 	<joint type="continuous" name="left_wheel_hinge">
-		<origin xyz="0 0.15 0" rpy="0 0 0"/>
+		<origin xyz="0 0.2 -0.05" rpy="0 0 0"/>
 		<child link="left_wheel"/>
 		<parent link="chassis"/>
@@ -112,5 +112,5 @@
 	</joint>
 	<joint type="continuous" name="right_wheel_hinge">
-		<origin xyz="0 -0.15 0" rpy="0 0 0"/>
+		<origin xyz="0 -0.2 -0.05" rpy="0 0 0"/>
 		<child link="right_wheel"/>
 		<parent link="chassis"/>
@@ -144,5 +144,5 @@
 	</link>
 	<joint name="camera_joint" type="fixed">
-		<origin xyz="0.2 0 0" rpy="0 0 0"/>
+		<origin xyz="0.15 0 0.1" rpy="0 0 0"/>
 		<child link="camera"/>
 		<parent link="chassis"/>
@@ -174,5 +174,5 @@
 	</link>
 	<joint name="hokuyo_joint" type="fixed">
-		<origin xyz="0.15 0 0.1" rpy="0 0 0"/>
+		<origin xyz="0.1 0 0.2" rpy="0 0 0"/>
 		<child link="hokuyo"/>
 		<parent link="chassis"/>
